Commit message: feat: update agv_robot package with gazebo worlds, config, and updated urdf

File: src/agv_robot/urdf/agv_robot_urdf.xacro (robot description, xacro)
@@ -61,5 +61,5 @@
     <visual>
       <geometry>
-        <cylinder radius="${platform_radius}" length="${platform_thickness}"/>
+        <box size="${2*platform_radius} ${wheel_track - wheel_width - 0.010} ${platform_thickness}"/>
       </geometry>
       <material name="dark_gray">
@@ -67,7 +67,9 @@
       </material>
     </visual>
+    <!-- collision: 바퀴(wheel_width/2 + 5mm 여유) 구간을 제외한 중앙 box로 근사 -->
+    <!-- Y폭 = 2 * (wheel_track/2 - wheel_width/2 - 0.005) = 0.219m -->
     <collision>
       <geometry>
-        <cylinder radius="${platform_radius}" length="${platform_thickness}"/>
+        <box size="${2*platform_radius} ${wheel_track - wheel_width - 0.010} ${platform_thickness}"/>
       </geometry>
     </collision>

Commit message: gazebo simul

File: src/agv_robot/urdf/agv_robot_urdf.xacro (robot description, xacro)
@@ -12,19 +12,23 @@
   <xacro:property name="wheel_track"   value="0.255"/>
   <!-- 지면 기준 절대 z → base_link 기준 상대 z 로 변환 시 wheel_radius 빼기 -->
-  <xacro:property name="lower_plate_z"  value="0.0225"/>  <!-- 0.020 + 0.005/2 -->
-  <xacro:property name="upper_plate_z"  value="0.0775"/>  <!-- 0.0225 + 0.050 + 0.005 -->
-  <xacro:property name="caster_radius"  value="0.0075"/>
-  <xacro:property name="caster_x"       value="0.130"/>
-  <xacro:property name="lidar_radius"   value="0.0482"/>
-  <xacro:property name="lidar_height"   value="0.0263"/>
-  <xacro:property name="camera_x"  value="0.148"/>
-  <xacro:property name="camera_z"  value="0.055"/>  <!-- ground 기준 -->
+  <xacro:property name="lower_plate_z" value="0.0225"/>   <!-- 0.020 + 0.005/2 -->
+  <xacro:property name="upper_plate_z" value="0.0775"/>   <!-- 0.0225 + 0.050 + 0.005 -->
+  <xacro:property name="caster_radius" value="0.0075"/>
+  <xacro:property name="caster_x"      value="0.130"/>
+  <xacro:property name="lidar_radius"  value="0.0482"/>
+  <xacro:property name="lidar_height"  value="0.0263"/>
+  <xacro:property name="camera_x"      value="0.148"/>
+  <xacro:property name="camera_z"      value="0.055"/>     <!-- ground 기준 -->
   <!-- ====================== INERTIA MACROS ==================== -->
   <xacro:macro name="inertia_cylinder" params="mass r l">
     <inertial>
       <mass value="${mass}"/>
-      <inertia ixx="${mass*(3*r*r+l*l)/12}" ixy="0" ixz="0"
-               iyy="${mass*(3*r*r+l*l)/12}" iyz="0"
-               izz="${mass*r*r/2}"/>
+      <inertia
+        ixx="${mass*(3*r*r+l*l)/12}"
+        ixy="0"
+        ixz="0"
+        iyy="${mass*(3*r*r+l*l)/12}"
+        iyz="0"
+        izz="${mass*r*r/2}"/>
     </inertial>
   </xacro:macro>
@@ -32,7 +36,11 @@
     <inertial>
       <mass value="${mass}"/>
-      <inertia ixx="${2*mass*r*r/5}" ixy="0" ixz="0"
-               iyy="${2*mass*r*r/5}" iyz="0"
-               izz="${2*mass*r*r/5}"/>
+      <inertia
+        ixx="${2*mass*r*r/5}"
+        ixy="0"
+        ixz="0"
+        iyy="${2*mass*r*r/5}"
+        iyz="0"
+        izz="${2*mass*r*r/5}"/>
     </inertial>
   </xacro:macro>
@@ -40,7 +48,11 @@
     <inertial>
       <mass value="${mass}"/>
-      <inertia ixx="${mass*(y*y+z*z)/12}" ixy="0" ixz="0"
-               iyy="${mass*(x*x+z*z)/12}" iyz="0"
-               izz="${mass*(x*x+y*y)/12}"/>
+      <inertia
+        ixx="${mass*(y*y+z*z)/12}"
+        ixy="0"
+        ixz="0"
+        iyy="${mass*(x*x+z*z)/12}"
+        iyz="0"
+        izz="${mass*(x*x+y*y)/12}"/>
     </inertial>
   </xacro:macro>
@@ -51,8 +63,10 @@
       <geometry><box size="0.001 0.001 0.001"/></geometry>
     </visual>
+    <!-- [추가] base_link inertial: Gazebo 자동 inertia 경고 방지용 더미 -->
+    <xacro:inertia_box mass="0.001" x="0.001" y="0.001" z="0.001"/>
   </link>
   <joint name="base_footprint_joint" type="fixed">
     <parent link="base_footprint"/>
-    <child  link="base_link"/>
+    <child link="base_link"/>
     <origin xyz="0 0 ${wheel_radius}" rpy="0 0 0"/>
   </joint>
@@ -61,5 +75,7 @@
     <visual>
       <geometry>
-        <box size="${2*platform_radius} ${wheel_track - wheel_width - 0.010} ${platform_thickness}"/>
+        <box size="${2*platform_radius}
+                   ${wheel_track - wheel_width - 0.010}
+                   ${platform_thickness}"/>
       </geometry>
       <material name="dark_gray">
@@ -71,12 +87,17 @@
     <collision>
       <geometry>
-        <box size="${2*platform_radius} ${wheel_track - wheel_width - 0.010} ${platform_thickness}"/>
+        <box size="${2*platform_radius}
+                   ${wheel_track - wheel_width - 0.010}
+                   ${platform_thickness}"/>
       </geometry>
     </collision>
-    <xacro:inertia_cylinder mass="0.8" r="${platform_radius}" l="${platform_thickness}"/>
+    <xacro:inertia_cylinder
+      mass="0.8"
+      r="${platform_radius}"
+      l="${platform_thickness}"/>
   </link>
   <joint name="lower_plate_joint" type="fixed">
     <parent link="base_link"/>
-    <child  link="lower_plate"/>
+    <child link="lower_plate"/>
     <origin xyz="0 0 ${lower_plate_z - wheel_radius}" rpy="0 0 0"/>
   </joint>
@@ -85,5 +106,6 @@
     <visual>
       <geometry>
-        <cylinder radius="${platform_radius}" length="${platform_thickness}"/>
+        <cylinder radius="${platform_radius}"
+                  length="${platform_thickness}"/>
       </geometry>
       <material name="dark_gray"/>
@@ -91,12 +113,16 @@
     <collision>
       <geometry>
-        <cylinder radius="${platform_radius}" length="${platform_thickness}"/>
+        <cylinder radius="${platform_radius}"
+                  length="${platform_thickness}"/>
       </geometry>
     </collision>
-    <xacro:inertia_cylinder mass="0.6" r="${platform_radius}" l="${platform_thickness}"/>
+    <xacro:inertia_cylinder
+      mass="0.6"
+      r="${platform_radius}"
+      l="${platform_thickness}"/>
   </link>
   <joint name="upper_plate_joint" type="fixed">
     <parent link="base_link"/>
-    <child  link="upper_plate"/>
+    <child link="upper_plate"/>
     <origin xyz="0 0 ${upper_plate_z - wheel_radius}" rpy="0 0 0"/>
   </joint>
@@ -106,5 +132,6 @@
       <visual>
         <geometry>
-          <cylinder radius="${wheel_radius}" length="${wheel_width}"/>
+          <cylinder radius="${wheel_radius}"
+                    length="${wheel_width}"/>
         </geometry>
         <material name="blue">
@@ -114,13 +141,19 @@
       <collision>
         <geometry>
-          <cylinder radius="${wheel_radius}" length="${wheel_width}"/>
+          <cylinder radius="${wheel_radius}"
+                    length="${wheel_width}"/>
         </geometry>
       </collision>
-      <xacro:inertia_cylinder mass="0.15" r="${wheel_radius}" l="${wheel_width}"/>
+      <xacro:inertia_cylinder
+        mass="0.15"
+        r="${wheel_radius}"
+        l="${wheel_width}"/>
     </link>
+    <!-- [수정] 휠축: 표준 설정으로 복원. cylinder 길이방향(Z)을 Y축으로 회전시킴 -->
     <joint name="${name}_joint" type="continuous">
       <parent link="base_link"/>
-      <child  link="${name}"/>
-      <origin xyz="0 ${side * wheel_track/2} 0" rpy="${pi/2} 0 0"/>
+      <child link="${name}"/>
+      <origin xyz="0 ${side * wheel_track/2} 0"
+              rpy="${pi/2} 0 0"/>
       <axis xyz="0 0 1"/>
       <dynamics damping="0.1" friction="0.1"/>
@@ -130,4 +163,6 @@
   <xacro:drive_wheel name="right_wheel" side="-1"/>
   <!-- ====================== BALL CASTERS ====================== -->
+  <!-- [수정] ball joint를 fixed → 2축 continuous로 변경 (자유 회전 허용)   -->
+  <!-- housing → (Y축 회전) → yaw_link → (X축 회전) → ball                  -->
   <xacro:macro name="ball_caster" params="name cx">
     <link name="${name}_housing">
@@ -136,10 +171,23 @@
         <material name="light_gray"><color rgba="0.7 0.7 0.7 1.0"/></material>
       </visual>
-      <xacro:inertia_box mass="0.02" x="0.02" y="0.02" z="0.01"/>
+      <xacro:inertia_box mass="0.01" x="0.02" y="0.02" z="0.01"/>
     </link>
     <joint name="${name}_housing_joint" type="fixed">
       <parent link="base_link"/>
-      <child  link="${name}_housing"/>
-      <origin xyz="${cx} 0 ${-wheel_radius + caster_radius + 0.005}" rpy="0 0 0"/>
+      <child link="${name}_housing"/>
+      <origin xyz="${cx} 0 ${-wheel_radius + caster_radius + 0.0075}"
+              rpy="0 0 0"/>
+    </joint>
+    <!-- [추가] 중간 더미 링크: 2축 자유 회전을 위한 가상 링크 -->
+    <link name="${name}_yaw_link">
+      <xacro:inertia_sphere mass="0.001" r="${caster_radius}"/>
+    </link>
+    <!-- 첫 번째 회전축: Z축 (좌우 미끄러짐 시 회전) -->
+    <joint name="${name}_yaw_joint" type="continuous">
+      <parent link="${name}_housing"/>
+      <child link="${name}_yaw_link"/>
+      <origin xyz="0 0 ${-caster_radius}" rpy="0 0 0"/>
+      <axis xyz="0 0 1"/>
+      <dynamics damping="0.0" friction="0.0"/>
     </joint>
     <link name="${name}_ball">
@@ -151,10 +199,13 @@
         <geometry><sphere radius="${caster_radius}"/></geometry>
       </collision>
-      <xacro:inertia_sphere mass="0.01" r="${caster_radius}"/>
+      <xacro:inertia_sphere mass="0.02" r="${caster_radius}"/>
     </link>
-    <joint name="${name}_ball_joint" type="fixed">
-      <parent link="${name}_housing"/>
-      <child  link="${name}_ball"/>
-      <origin xyz="0 0 ${-caster_radius}" rpy="0 0 0"/>
+    <!-- 두 번째 회전축: X축 (전후진 시 굴러감) -->
+    <joint name="${name}_ball_joint" type="continuous">
+      <parent link="${name}_yaw_link"/>
+      <child link="${name}_ball"/>
+      <origin xyz="0 0 0" rpy="0 0 0"/>
+      <axis xyz="1 0 0"/>
+      <dynamics damping="0.0" friction="0.0"/>
     </joint>
   </xacro:macro>
@@ -165,5 +216,6 @@
     <visual>
       <geometry>
-        <cylinder radius="${lidar_radius}" length="${lidar_height}"/>
+        <cylinder radius="${lidar_radius}"
+                  length="${lidar_height}"/>
       </geometry>
       <material name="black"><color rgba="0.1 0.1 0.1 1.0"/></material>
@@ -171,13 +223,18 @@
     <collision>
       <geometry>
-        <cylinder radius="${lidar_radius}" length="${lidar_height}"/>
+        <cylinder radius="${lidar_radius}"
+                  length="${lidar_height}"/>
       </geometry>
     </collision>
-    <xacro:inertia_cylinder mass="0.17" r="${lidar_radius}" l="${lidar_height}"/>
+    <xacro:inertia_cylinder
+      mass="0.17"
+      r="${lidar_radius}"
+      l="${lidar_height}"/>
   </link>
   <joint name="lidar_joint" type="fixed">
     <parent link="upper_plate"/>
-    <child  link="lidar_link"/>
-    <origin xyz="0 0 ${platform_thickness/2 + lidar_height/2}" rpy="0 0 0"/>
+    <child link="lidar_link"/>
+    <origin xyz="0 0 ${platform_thickness/2 + lidar_height/2}"
+            rpy="0 0 0"/>
   </joint>
   <!-- ======================== CAMERA ========================== -->
@@ -194,6 +251,7 @@
   <joint name="camera_joint" type="fixed">
     <parent link="base_link"/>
-    <child  link="camera_link"/>
-    <origin xyz="${camera_x} 0 ${camera_z - wheel_radius}" rpy="0 0 0"/>
+    <child link="camera_link"/>
+    <origin xyz="${camera_x} 0 ${camera_z - wheel_radius}"
+            rpy="0 0 0"/>
   </joint>
   <!-- camera_optical_frame: ROS 카메라 좌표계 (Z-forward) -->
@@ -201,5 +259,5 @@
   <joint name="camera_optical_joint" type="fixed">
     <parent link="camera_link"/>
-    <child  link="camera_optical_frame"/>
+    <child link="camera_optical_frame"/>
     <origin xyz="0 0 0" rpy="${-pi/2} 0 ${-pi/2}"/>
   </joint>
@@ -207,6 +265,7 @@
   <!-- 차동구동 -->
   <gazebo>
-    <plugin filename="gz-sim-diff-drive-system"
-            name="gz::sim::systems::DiffDrive">
+    <plugin
+      filename="gz-sim-diff-drive-system"
+      name="gz::sim::systems::DiffDrive">
       <left_joint>left_wheel_joint</left_joint>
       <right_joint>right_wheel_joint</right_joint>
@@ -223,31 +282,23 @@
   <!-- 볼캐스터 마찰 제거 -->
   <gazebo reference="front_caster_ball">
-    <surface>
-      <friction>
-        <ode><mu>0</mu><mu2>0</mu2></ode>
-      </friction>
-    </surface>
+    <mu1>0.0</mu1>
+    <mu2>0.0</mu2>
   </gazebo>
   <gazebo reference="rear_caster_ball">
-    <surface>
-      <friction>
-        <ode><mu>0</mu><mu2>0</mu2></ode>
-      </friction>
-    </surface>
-  </gazebo>
-  <!-- 바퀴 마찰 -->
+    <mu1>0.0</mu1>
+    <mu2>0.0</mu2>
+  </gazebo>
+  <!-- [수정] 바퀴 마찰: mu1=2.0, mu2=0.2 (이전 메시지 값) -->
   <gazebo reference="left_wheel">
-    <surface>
-      <friction>
-        <ode><mu>1.0</mu><mu2>0.5</mu2></ode>
-      </friction>
-    </surface>
+    <mu1>1.0</mu1>
+    <mu2>1.0</mu2>
+    <kp>1e6</kp>
+    <kd>1.0</kd>
   </gazebo>
   <gazebo reference="right_wheel">
-    <surface>
-      <friction>
-        <ode><mu>1.0</mu><mu2>0.5</mu2></ode>
-      </friction>
-    </surface>
+    <mu1>1.0</mu1>
+    <mu2>1.0</mu2>
+    <kp>1e6</kp>
+    <kd>1.0</kd>
   </gazebo>
   <!-- LiDAR 센서 : LDROBOT D200 (LD14P) -->
@@ -289,5 +340,5 @@
       <update_rate>30</update_rate>
       <camera>
-        <horizontal_fov>1.2217</horizontal_fov>  <!-- 70° -->
+        <horizontal_fov>1.2217</horizontal_fov>   <!-- 70° -->
         <image>
           <width>1280</width>
